Commit message: med14 -> med14_r820

File: urdf/med14_r820.urdf.xacro (robot description, xacro)
@@ -2,13 +2,13 @@
 <!-- top level -->
 <robot name="med14" xmlns:xacro="http://www.ros.org/wiki/xacro">
-    <!-- include the med14 macro -->
-    <xacro:include filename="$(find med14_description)/urdf/med14_macro.xacro" />
+    <!-- include the Med 14 R820 macro -->
+    <xacro:include filename="$(find med14_r820_description)/urdf/med14_r820_macro.xacro" />
     <!-- arguments -->
     <xacro:arg name="robot_name" default="lbr" />
     <xacro:arg
         name="joint_limits_path"
-        default="$(find med14_description)/config/joint_limits.yaml" />
-    <!-- med14 description -->
-    <xacro:med14
+        default="$(find med14_r820_description)/config/joint_limits.yaml" />
+    <!-- Med 14 R820 description -->
+    <xacro:med14_r820
         robot_name="$(arg robot_name)"
         joint_limits_path="$(arg joint_limits_path)" />

File: urdf/med14_r820_macro.xacro (robot description, xacro)
@@ -2,6 +2,6 @@
 <root xmlns:xacro="http://www.ros.org/wiki/xacro">
     <!-- robot as extracted via https://github.com/syuntoku14/fusion2urdf -->
-    <xacro:macro name="med14"
-        params="robot_name:=^|lbr joint_limits_path:=^|'$(find med14_description)/config/joint_limits.yaml'">
+    <xacro:macro name="med14_r820"
+        params="robot_name:=^|lbr joint_limits_path:=^|'$(find med14_r820_description)/config/joint_limits.yaml'">
         <!-- load joint limits via yaml -->
         <xacro:property name="joint_limits" value="${xacro.load_yaml(joint_limits_path)}" />
@@ -21,5 +21,5 @@
                 <origin rpy="0 0 0" xyz="0 0 0" />
                 <geometry>
-                    <mesh filename="package://med14_description/meshes/visual/link_0.dae" />
+                    <mesh filename="package://med14_r820_description/meshes/visual/link_0.dae" />
                 </geometry>
             </visual>
@@ -27,5 +27,5 @@
                 <origin rpy="0 0 0" xyz="0 0 0" />
                 <geometry>
-                    <mesh filename="package://med14_description/meshes/collision/link_0.stl" />
+                    <mesh filename="package://med14_r820_description/meshes/collision/link_0.stl" />
                 </geometry>
             </collision>
@@ -58,5 +58,5 @@
                 <origin rpy="0 0 0" xyz="0.0 0.0 -0.147" />
                 <geometry>
-                    <mesh filename="package://med14_description/meshes/visual/link_1.dae" />
+                    <mesh filename="package://med14_r820_description/meshes/visual/link_1.dae" />
                 </geometry>
             </visual>
@@ -64,5 +64,5 @@
                 <origin rpy="0 0 0" xyz="0.0 0.0 -0.147" />
                 <geometry>
-                    <mesh filename="package://med14_description/meshes/collision/link_1.stl" />
+                    <mesh filename="package://med14_r820_description/meshes/collision/link_1.stl" />
                 </geometry>
             </collision>
@@ -95,5 +95,5 @@
                 <origin rpy="0 0 0" xyz="0.0 0.01 -0.3595" />
                 <geometry>
-                    <mesh filename="package://med14_description/meshes/visual/link_2.dae" />
+                    <mesh filename="package://med14_r820_description/meshes/visual/link_2.dae" />
                 </geometry>
             </visual>
@@ -101,5 +101,5 @@
                 <origin rpy="0 0 0" xyz="0.0 0.01 -0.3595" />
                 <geometry>
-                    <mesh filename="package://med14_description/meshes/collision/link_2.stl" />
+                    <mesh filename="package://med14_r820_description/meshes/collision/link_2.stl" />
                 </geometry>
             </collision>
@@ -132,5 +132,5 @@
                 <origin rpy="0 0 0" xyz="0.0 0.0 -0.5875" />
                 <geometry>
-                    <mesh filename="package://med14_description/meshes/visual/link_3.dae" />
+                    <mesh filename="package://med14_r820_description/meshes/visual/link_3.dae" />
                 </geometry>
             </visual>
@@ -138,5 +138,5 @@
                 <origin rpy="0 0 0" xyz="0.0 0.0 -0.5875" />
                 <geometry>
-                    <mesh filename="package://med14_description/meshes/collision/link_3.stl" />
+                    <mesh filename="package://med14_r820_description/meshes/collision/link_3.stl" />
                 </geometry>
             </collision>
@@ -169,5 +169,5 @@
                 <origin rpy="0 0 0" xyz="0.0 -0.0105 -0.7795" />
                 <geometry>
-                    <mesh filename="package://med14_description/meshes/visual/link_4.dae" />
+                    <mesh filename="package://med14_r820_description/meshes/visual/link_4.dae" />
                 </geometry>
             </visual>
@@ -175,5 +175,5 @@
                 <origin rpy="0 0 0" xyz="0.0 -0.0105 -0.7795" />
                 <geometry>
-                    <mesh filename="package://med14_description/meshes/collision/link_4.stl" />
+                    <mesh filename="package://med14_r820_description/meshes/collision/link_4.stl" />
                 </geometry>
             </collision>
@@ -206,5 +206,5 @@
                 <origin rpy="0 0 0" xyz="0.0 0.0 -0.987" />
                 <geometry>
-                    <mesh filename="package://med14_description/meshes/visual/link_5.dae" />
+                    <mesh filename="package://med14_r820_description/meshes/visual/link_5.dae" />
                 </geometry>
             </visual>
@@ -212,5 +212,5 @@
                 <origin rpy="0 0 0" xyz="0.0 0.0 -0.987" />
                 <geometry>
-                    <mesh filename="package://med14_description/meshes/collision/link_5.stl" />
+                    <mesh filename="package://med14_r820_description/meshes/collision/link_5.stl" />
                 </geometry>
             </collision>
@@ -243,5 +243,5 @@
                 <origin rpy="0 0 0" xyz="0.0 0.0707 -1.1795" />
                 <geometry>
-                    <mesh filename="package://med14_description/meshes/visual/link_6.dae" />
+                    <mesh filename="package://med14_r820_description/meshes/visual/link_6.dae" />
                 </geometry>
             </visual>
@@ -249,5 +249,5 @@
                 <origin rpy="0 0 0" xyz="0.0 0.0707 -1.1795" />
                 <geometry>
-                    <mesh filename="package://med14_description/meshes/collision/link_6.stl" />
+                    <mesh filename="package://med14_r820_description/meshes/collision/link_6.stl" />
                 </geometry>
             </collision>
@@ -279,5 +279,5 @@
                 <origin rpy="0 0 0" xyz="0.0 0.0 -1.2705" />
                 <geometry>
-                    <mesh filename="package://med14_description/meshes/visual/link_7.dae" />
+                    <mesh filename="package://med14_r820_description/meshes/visual/link_7.dae" />
                 </geometry>
             </visual>
@@ -285,5 +285,5 @@
                 <origin rpy="0 0 0" xyz="0.0 0.0 -1.2705" />
                 <geometry>
-                    <mesh filename="package://med14_description/meshes/collision/link_7.stl" />
+                    <mesh filename="package://med14_r820_description/meshes/collision/link_7.stl" />
                 </geometry>
             </collision>
